Commit message: Ur5 reach working, tested with DDPG and SAC

File: UR_gym/envs/robots/urdf/ur5.urdf (robot description, URDF)
Before this commit: robot universal_robot, 8 links, 7 joints
Links:
- link base_link: geometry collision mesh filename=../meshes/ur5/collision/base.stl; visual mesh filename=../meshes/ur5/visual/base.obj
- link forearm_link: geometry collision mesh filename=../meshes/ur5/collision/forearm.stl; visual mesh filename=../meshes/ur5/visual/forearm.obj
- link shoulder_link: geometry collision mesh filename=../meshes/ur5/collision/shoulder.stl; visual mesh filename=../meshes/ur5/visual/shoulder.obj
- link upper_arm_link: geometry collision mesh filename=../meshes/ur5/collision/upperarm.stl; visual mesh filename=../meshes/ur5/visual/upperarm.obj
- link wrist_1_link: geometry collision mesh filename=../meshes/ur5/collision/wrist1.stl; visual mesh filename=../meshes/ur5/visual/wrist1.obj
- link wrist_2_link: geometry collision mesh filename=../meshes/ur5/collision/wrist2.stl; visual mesh filename=../meshes/ur5/visual/wrist2.obj
- link wrist_3_link: geometry collision mesh filename=../meshes/ur5/collision/wrist3.stl; visual mesh filename=../meshes/ur5/visual/wrist3.obj
Joints:
- joint shoulder_lift_joint: limit lower=-6.28318530718 upper=6.28318530718 effort=150.0 velocity=3.15 -> lower=-3.14159265359 upper=3.14159265359 effort=150.0 velocity=3.15
- joint shoulder_pan_joint: limit lower=-6.28318530718 upper=6.28318530718 effort=150.0 velocity=3.15 -> lower=-3.14159265359 upper=3.14159265359 effort=150.0 velocity=3.15
- joint wrist_1_joint: limit lower=-6.28318530718 upper=6.28318530718 effort=28.0 velocity=3.2 -> lower=-3.14159265359 upper=3.14159265359 effort=28.0 velocity=3.2
- joint wrist_2_joint: limit lower=-6.28318530718 upper=6.28318530718 effort=28.0 velocity=3.2 -> lower=-3.14159265359 upper=3.14159265359 effort=28.0 velocity=3.2
- joint wrist_3_joint: limit lower=-6.28318530718 upper=6.28318530718 effort=28.0 velocity=3.2 -> lower=-3.14159265359 upper=3.14159265359 effort=28.0 velocity=3.2

Commit message: UR5 on workbench working, verified with SAC

File: UR_gym/envs/robots/urdf/ur5.urdf (robot description, URDF)
Before this commit: robot universal_robot, 8 links, 7 joints
Links:
- link base_link: geometry collision mesh filename=../meshes/ur5/collision/base.stl; visual mesh filename=../meshes/ur5/visual/base.dae
- link forearm_link: geometry collision mesh filename=../meshes/ur5/collision/forearm.stl; visual mesh filename=../meshes/ur5/visual/forearm.dae
- link shoulder_link: geometry collision mesh filename=../meshes/ur5/collision/shoulder.stl; visual mesh filename=../meshes/ur5/visual/shoulder.dae
- link upper_arm_link: geometry collision mesh filename=../meshes/ur5/collision/upperarm.stl; visual mesh filename=../meshes/ur5/visual/upperarm.dae
- link wrist_1_link: geometry collision mesh filename=../meshes/ur5/collision/wrist1.stl; visual mesh filename=../meshes/ur5/visual/wrist1.dae
- link wrist_2_link: geometry collision mesh filename=../meshes/ur5/collision/wrist2.stl; visual mesh filename=../meshes/ur5/visual/wrist2.dae
- link wrist_3_link: geometry collision mesh filename=../meshes/ur5/collision/wrist3.stl; visual mesh filename=../meshes/ur5/visual/wrist3.dae
