Commit message: the pybullet ik solver is bad, trying to use the ikfast package. Replaced ur5 with ur5e

File: UR_gym/envs/robots/urdf/ur5e.urdf (robot description, URDF)
Before this commit: robot ur5e_robot, 11 links, 10 joints
Links:
- removed link flange
- removed link tool0
- added link ee_link; collision box size=0.01 0.01 0.01
- link base_link_inertia: geometry collision mesh filename=../meshes/ur5/collision/base.stl; visual mesh filename=../meshes/ur5/visual/base.dae
- link forearm_link: geometry collision mesh filename=../meshes/ur5/collision/forearm.stl; visual mesh filename=../meshes/ur5/visual/forearm.dae
- link shoulder_link: geometry collision mesh filename=../meshes/ur5/collision/shoulder.stl; visual mesh filename=../meshes/ur5/visual/shoulder.dae
- link upper_arm_link: geometry collision mesh filename=../meshes/ur5/collision/upperarm.stl; visual mesh filename=../meshes/ur5/visual/upperarm.dae
- link wrist_1_link: geometry collision mesh filename=../meshes/ur5/collision/wrist1.stl; visual mesh filename=../meshes/ur5/visual/wrist1.dae
- link wrist_2_link: geometry collision mesh filename=../meshes/ur5/collision/wrist2.stl; visual mesh filename=../meshes/ur5/visual/wrist2.dae
- link wrist_3_link: geometry collision mesh filename=../meshes/ur5/collision/wrist3.stl; visual mesh filename=../meshes/ur5/visual/wrist3.dae
Joints:
- removed joint flange-tool0
- removed joint wrist_3-flange
- added joint ee_fixed_joint: type fixed, parent wrist_3_link, child ee_link, origin xyz=0.0 0.0 0.0 rpy=0.0 0.0 1.57079632679

Commit message: Adding goal checking code using inverse kinematics

File: UR_gym/envs/robots/urdf/ur5e.urdf (robot description, URDF)
Before this commit: robot ur5e_robot, 10 links, 9 joints
Joints:
- joint ee_fixed_joint: origin xyz=0.0 0.0 0.0 rpy=0.0 0.0 1.57079632679 -> xyz=0.0 0.0 0.0 rpy=0.0 0.0 0.0
